File: RobomasSwerve.sch (EAGLE design)
At the start: 50 parts, among them J1 8P8C-LED, J2 XT60PW-M, J3 MA04-1, J4 10118192-0001LF, J5 EP2.5-4-SIDE, U1 STM32F302C, U2 NCV7351D1E, U3 SI8621AB-B-IS, U4 AP2127N-3.3TRG1, U5 78L05F, U6 TLP291, X1 CSTCE8M00G55

Commit message: update
Parts:
- removed U$1: XH-2-STRAIGHT, con-xh:XH-2-STRAIGHT
- added J10, J11, J12, J13, J14, J15, J9: BM02B-GHS-TBT_LF__SN_, BM02B-GHS-TBT_LF__SN_:BM02B-GHS-TBT_LF__SN_
- added J6, J7, J8: EP2.5-4-SIDE, con-ep2.5:EP2.5-4-SIDE
- J2: value XT60PW-M -> BM02B-GHS-TBT_LF__SN_; device con-xt:XT60PW-M -> BM02B-GHS-TBT_LF__SN_:BM02B-GHS-TBT_LF__SN_
Connections:
- removed net ENC_A: J5.3
- removed net ENC_B: J5.4
- net !EMS: now also U1.PC13-TAMPER-RTC; no longer U1.PB5
- net +12V: now also C1.+; no longer J1.4, J1.5, J1.A-G
- net +5V: now also J6.2, J7.2, J8.2
- net +5V_ISO: no longer U$1.2
- net CANH: now also J10.2, J11.2, J12.2, J13.2, J14.2, J15.2, J2.2, J9.2
- net CANL: now also J10.1, J11.1, J12.1, J13.1, J14.1, J15.1, J2.1, J9.1
- net CAN_LED: now also U1.VBAT; no longer U1.PB4-JNTRST
- net DCIN: now also J1.4, J1.5, J1.A-G; no longer C1.+, J2.2
- net EMS: no longer U$1.1
- net GNDA: now also J6.1, J7.1, J8.1
- net GNDIO: no longer J2.GND
- net LED0: now also U1.PB0
- net LED1: now also U1.PB1
- net LED2: now also U1.PB2
- net TIM1_CH1: now also J5.3
- net TIM1_CH2: now also J5.4
- net TIM2_CH1: now also J7.3
- net TIM2_CH2: now also J7.4
- net TIM3_CH1: now also J6.4
- net TIM3_CH2: now also J6.3
- net TIM4_CH1: now also J8.3
- net TIM4_CH2: now also J8.4
Other:
- moved on the sheet: F1, J2, J5
